File: PCBshield/FoamBot Arduino Pololu servo r1.brd (EAGLE design)
At the start: 71.1 x 59.4 mm, 19 parts, among them U1 ARDUINO_SHIELDLABEL, U2 POLOLU_A4983CARRIER, U3 POLOLU_A4983CARRIER, X1 MSTBA2, X4 22-23-2021, X5 22-23-2031

Commit message: cleaned up pcb
Parts:
- moved C5 0.64 mm to (74.3, 27.9)
Routing:
- net N$5: track 0.00 -> 17.0 mm
- net GND: track 140.9 -> 150.1 mm
- net VCC: track 149.8 -> 147.3 mm
- net +12V: track 143.7 -> 143.0 mm
Changed lines of the file:
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@@
 <wire x1="79.99" y1="59.36" x2="8.89" y2="59.36" width="0" layer="20"/>
 <wire x1="8.89" y1="59.36" x2="8.89" y2="0" width="0" layer="20"/>
-<rectangle x1="11.43" y1="30.48" x2="31.75" y2="50.8" layer="1"/>
+<rectangle x1="11.43" y1="30.48" x2="31.75" y2="50.8" layer="121"/>
 </plain>
 <attributes>
@@
 </element>
 <element name="C3" library="capacitor-wima" package="C2.5-3" value="100nF" x="51.435" y="27.305" rot="R90"/>
-<element name="C5" library="capacitor-wima" package="C2.5-3" value="100nF" x="73.66" y="27.94" rot="R90"/>
+<element name="C5" library="capacitor-wima" package="C2.5-3" value="100nF" x="74.295" y="27.94" rot="R90"/>
 </elements>
 <signals>
@@
 <wire x1="59.69" y1="29.21" x2="60.96" y2="30.48" width="1.016" layer="16"/>
 <wire x1="60.96" y1="30.48" x2="60.96" y2="32.385" width="1.016" layer="16"/>
-<wire x1="38.1" y1="32.385" x2="38.1" y2="31.115" width="1.016" layer="16"/>
-<via x="38.1" y="31.115" extent="1-16" drill="0.6" diameter="1.27"/>
-<wire x1="38.1" y1="31.115" x2="38.1" y2="38.735" width="1.016" layer="1"/>
+<wire x1="38.1" y1="32.385" x2="38.1" y2="33.655" width="1.016" layer="16"/>
+<via x="38.1" y="33.655" extent="1-16" drill="0.6" diameter="1.27"/>
+<wire x1="38.1" y1="33.655" x2="38.1" y2="38.735" width="1.016" layer="1"/>
 <contactref element="U2" pad="MS3"/>
 <contactref element="JP2" pad="5"/>
@@
 </signal>
 <signal name="N$7">
-<via x="60.96" y="31.115" extent="1-16" drill="0.6" diameter="1.27"/>
+<via x="60.96" y="33.655" extent="1-16" drill="0.6" diameter="1.27"/>
 </signal>
 <signal name="N$3">
@@
 <contactref element="C5" pad="1"/>
 <wire x1="51.435" y1="26.035" x2="53.34" y2="26.035" width="1.016" layer="16"/>
-<via x="53.34" y="26.035" extent="1-16" drill="0.6" shape="square"/>
-<wire x1="73.66" y1="26.67" x2="76.2" y2="26.67" width="1.016" layer="16"/>
+<via x="53.34" y="26.035" extent="1-16" drill="0.6" diameter="1.27"/>
+<wire x1="74.295" y1="26.67" x2="76.2" y2="26.67" width="1.016" layer="16"/>
 </signal>
 <signal name="GND">
@@
 <wire x1="19.05" y1="53.34" x2="22.86" y2="49.53" width="1.016" layer="16"/>
 <wire x1="22.86" y1="49.53" x2="31.75" y2="49.53" width="1.016" layer="16"/>
-<wire x1="35.56" y1="53.34" x2="35.56" y2="49.53" width="1.016" layer="16"/>
-<wire x1="35.56" y1="49.53" x2="31.75" y2="49.53" width="1.016" layer="16"/>
+<wire x1="35.56" y1="53.34" x2="35.56" y2="51.32605" width="1.016" layer="16"/>
+<wire x1="35.56" y1="51.32605" x2="33.76395" y2="49.53" width="1.016" layer="16"/>
+<wire x1="33.76395" y1="49.53" x2="31.75" y2="49.53" width="1.016" layer="16"/>
 <wire x1="31.75" y1="49.53" x2="31.75" y2="38.735" width="1.016" layer="16"/>
 <wire x1="31.75" y1="38.735" x2="35.56" y2="36.195" width="1.016" layer="16"/>
@@
 <contactref element="C3" pad="2"/>
 <contactref element="C5" pad="2"/>
+<wire x1="74.295" y1="29.21" x2="74.295" y2="29.845" width="1.016" layer="16"/>
+<wire x1="74.295" y1="29.845" x2="73.66" y2="30.48" width="1.016" layer="16"/>
+<wire x1="73.66" y1="30.48" x2="73.66" y2="32.385" width="1.016" layer="16"/>
+<wire x1="51.435" y1="28.575" x2="51.435" y2="29.21" width="1.016" layer="16"/>
+<wire x1="51.435" y1="29.21" x2="50.8" y2="29.845" width="1.016" layer="16"/>
+<wire x1="50.8" y1="29.845" x2="50.8" y2="32.385" width="1.016" layer="16"/>
+<wire x1="52.07" y1="4.445" x2="50.165" y2="4.445" width="1.016" layer="16"/>
+<wire x1="50.165" y1="4.445" x2="49.53" y2="5.08" width="1.016" layer="16"/>
 </signal>
 <signal name="N$1">
@@
 <wire x1="49.53" y1="19.05" x2="50.8" y2="19.05" width="1.016" layer="16"/>
 </signal>
+<signal name="N$5">
+<wire x1="19.685" y1="11.43" x2="22.225" y2="11.43" width="1.016" layer="16"/>
+<wire x1="22.225" y1="11.43" x2="27.305" y2="6.35" width="1.016" layer="16"/>
+<wire x1="27.305" y1="6.35" x2="33.655" y2="6.35" width="1.016" layer="16"/>
+<wire x1="33.655" y1="6.35" x2="34.29" y2="5.715" width="1.016" layer="16"/>
+</signal>
 </signals>
